File: KeyboardController.kicad_pcb (KiCad board)
At the start: 2 copper layers, 40.6 x 49.5 mm, 11 parts, among them J1 KMDGX-6S-BS, J2 KMDGX-6S-BS, J3 HDR_D, J4 HDR_S, U1 ATtiny461A-P, U2 74HC164, Y1 ECS-080-20-4X-DU

Commit message: Board rev 1.
Parts:
- added C5: 100n, Capacitor_THT:C_Rect_L4.0mm_W2.5mm_P2.50mm, F.Cu at (165.6, 100.2)
- J2: value KMDGX-6S-BS -> HDR_ISP; footprint KiCad:KMDGX6SBS -> Connector_PinHeader_2.54mm:PinHeader_2x03_P2.54mm_Vertical
- moved J3 42.3 mm to (146.1, 110.7), turned to 0 degrees
- moved J4 42.3 mm to (181.6, 110.7), turned to 0 degrees
- moved J2 29.3 mm to (147.1, 118.9), turned to 90 degrees
- moved C2 2.30 mm to (173.5, 115.2)
- moved U1 2.22 mm to (152.9, 111.4)
- moved Y1 2.22 mm to (171.9, 120.3)
- moved C1 2.22 mm to (165.6, 115.2)
- moved C3 2.22 mm to (163.1, 115.2)
- moved C4 1.18 mm to (154.0, 87.7)
- moved U2 1.18 mm to (157.8, 95.4)
Connections:
- net /IRQB renamed /PA4
- J2 pad 1: /PS2B_DATA -> /MISO
- J2 pad 2: unconnected-(J2-Pad2) -> +5V
- J2 pad 3: GND -> /SCK
- J2 pad 5: +5V -> /~{RST}
- J2 pad 6: /PS2B_CLK -> GND
- J4 pad 7: /PB7 -> unconnected-(J4-Pad7)
- J4 pad 8: /PB6 -> unconnected-(J4-Pad8)
- U1 pad 1: /PS2A_CLK -> /MOSI
- U1 pad 10: /PB7 -> /~{RST}
- U1 pad 2: /PS2A_DATA -> /MISO
- U1 pad 3: /PS2B_CLK -> /SCK
- U1 pad 4: /PS2B_DATA -> /PS2A_CLK
- U1 pad 9: /PB6 -> /PS2A_DATA
Routing:
- net GND: track 53.5 -> 0.00 mm
- net /PS2B_CLK: track 32.4 -> 0.00 mm, vias 2 -> 0
- net /PB7: track 31.7 -> 0.00 mm, vias 2 -> 0
- net /PS2B_DATA: track 31.5 -> 0.00 mm
- net /~{RST}: track 0.00 -> 31.0 mm
- net /PB6: track 28.1 -> 0.00 mm, vias 2 -> 0
- net /PA7: track 32.1 -> 8.07 mm, vias 2 -> 0
- net +5V: track 149.8 -> 131.9 mm, vias 2 -> 0
- net /PA4: track 32.9 -> 15.1 mm
- net /D7: track 33.9 -> 16.3 mm
- net /PA6: track 28.1 -> 11.0 mm, vias 1 -> 0
- net /PS2A_DATA: track 17.8 -> 34.0 mm
- net /D3: track 12.1 -> 27.9 mm
- net /PA5: track 27.0 -> 13.1 mm, vias 2 -> 0
- net /SCK: track 0.00 -> 12.8 mm
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Other:
- board text added: "8Mhz"
- board text added: "IRQ"
- board text added: "ISP"
- board text added: "PA4"
- board text added: "Rev 1"
- board text added: "© microcode.io"
- board text removed: "IRQA"
- board text removed: "IRQB"
- board text removed: "PB6"
- board text removed: "PB7"
- board text removed: "Rev 0"
