File: KeyboardController.kicad_sch (KiCad schematic)
At the start: 11 parts, among them J1 KMDGX-6S-BS, J2 KMDGX-6S-BS, J3 HDR_D, J4 HDR_S, U1 ATtiny461A-P, U2 74HC164, Y1 ECS-080-20-4X-DU

Commit message: Board rev 1.
Parts:
- removed J2: KMDGX-6S-BS, KiCad:KMDGX6SBS, symbol KMDGX-6S-BS:KMDGX-6S-BS
- added C5: 100n, Capacitor_THT:C_Rect_L4.0mm_W2.5mm_P2.50mm, symbol Device:C_Small
- added J2: HDR_ISP, Connector_PinHeader_2.54mm:PinHeader_2x03_P2.54mm_Vertical, symbol Connector_Generic:Conn_02x03_Odd_Even
Connections:
- net PS2B_DATA is gone; now on net PS2A_CLK: U1.4 (PB3)
- net +5V: now also C5.1, J2.2 (Pin_2)
- net GND: now also C5.2, J2.6 (Pin_6)
- net PS2A_CLK: no longer U1.1 (PB0)
- net PS2A_DATA: now also U1.9 (PB6); no longer U1.2 (PB1)
- net IRQB renamed PA4
- net PB6: no longer names the net of J4.8 (Pin_8)
- net PB6: no longer U1.9 (PB6)
- net PB7: no longer names the net of J4.7 (Pin_7)
- net PB7: no longer U1.10 (~{RESET}/PB7)
- net PS2B_CLK renamed SCK
- net SCK: now also J2.3 (Pin_3)
- new net MISO: J2.1 (Pin_1), U1.2 (PB1)
- new net MOSI: J2.4 (Pin_4), U1.1 (PB0)
- new net ~{RST}: J2.5 (Pin_5), U1.10 (~{RESET}/PB7)
Other:
- company: (none) -> Microcode.io
- title: (none) -> PS/2 Keyboard Serial to Parallel Interface
